Commit message: Fixed bad collision meshes, corrupted objects

File: urdf/office_extension_geometry.urdf.xacro (robot description, xacro)
@@ -1,5 +1,5 @@
 <?xml version="1.0"?>
-<robot name="office_world" xmlns:xacro="http://www.ros.org/wiki/xacro">
-  <link name="office_world_link">
+<robot name="office_extension_world" xmlns:xacro="http://www.ros.org/wiki/xacro">
+  <link name="office_world_extension_link">
     <inertial>
       <origin xyz="0 0 0" rpy="0 0 0"/>
